File: Schematics/nucleo.kicad_sch (KiCad schematic)
At the start: 5 parts, among them U1 NUCLEO144-F767ZI

Commit message: Moved all Nucleo connections to one side of the board
Connections:
- net at U1.109 (PA3): now also R2.2, R3.1
- net at U1.38 (PC0): now also R1.1
- net at U1.94 (PB2): no longer R1.1
- now unconnected: U1.96 (PB1)
Changed lines of the file:
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@@
   (no_connect (at 50.8 71.12))
   (no_connect (at 66.04 71.12))
-  (no_connect (at 55.88 71.12))
   (no_connect (at 215.9 71.12))
   (no_connect (at 177.8 137.16))
@@
   (no_connect (at 200.66 71.12))
   (no_connect (at 228.6 121.92))
+  (no_connect (at 93.98 71.12))
   (no_connect (at 228.6 93.98))
   (no_connect (at 48.26 137.16))
@@
   (no_connect (at 142.24 71.12))
   (no_connect (at 213.36 137.16))
-  (no_connect (at 134.62 71.12))
   (no_connect (at 172.72 71.12))
   (no_connect (at 228.6 116.84))
@@
   (no_connect (at 127 71.12))
   (no_connect (at 203.2 71.12))
+  (no_connect (at 96.52 71.12))
   (no_connect (at 76.2 71.12))
   (no_connect (at 60.96 71.12))
@@
   (no_connect (at 53.34 71.12))
   (no_connect (at 104.14 71.12))
-  (wire (pts (xy 252.73 83.82) (xy 257.81 83.82))
+  (wire (pts (xy 134.62 67.31) (xy 245.11 67.31))
     (stroke (width 0) (type default) (color 0 0 0 0))
   )
-  (wire (pts (xy 93.98 71.12) (xy 93.98 63.5))
+  (wire (pts (xy 252.73 83.82) (xy 257.81 83.82))
     (stroke (width 0) (type default) (color 0 0 0 0))
   )
@@
     (stroke (width 0) (type default) (color 0 0 0 0))
   )
-  (wire (pts (xy 93.98 63.5) (xy 252.73 63.5))
+  (wire (pts (xy 55.88 71.12) (xy 55.88 63.5))
     (stroke (width 0) (type default) (color 0 0 0 0))
   )
@@
     (stroke (width 0) (type default) (color 0 0 0 0))
   )
+  (wire (pts (xy 55.88 63.5) (xy 252.73 63.5))
+    (stroke (width 0) (type default) (color 0 0 0 0))
+  )
   (wire (pts (xy 245.11 91.44) (xy 245.11 82.55))
+    (stroke (width 0) (type default) (color 0 0 0 0))
+  )
+  (wire (pts (xy 134.62 71.12) (xy 134.62 67.31))
     (stroke (width 0) (type default) (color 0 0 0 0))
   )
@@
     (stroke (width 0) (type default) (color 0 0 0 0))
   )
-  (wire (pts (xy 96.52 67.31) (xy 96.52 71.12))
-    (stroke (width 0) (type default) (color 0 0 0 0))
-  )
-  (wire (pts (xy 245.11 67.31) (xy 96.52 67.31))
-    (stroke (width 0) (type default) (color 0 0 0 0))
-  )
